File: aoi bara_青いバラ/pcb/pcb/_autosave-pcb.kicad_pcb (KiCad board)
At the start: 2 copper layers, 314.3 x 95.2 mm, 136 parts, among them J1 OLED_128x64, U1 Raspberry_Pi_Pico

Commit message: deleted:    "aoi bara_\351\235\222\343\201\204\343\203\220\343\203\251/frimware/aoi_bara/aoi_bara.c" 	modified:   "aoi bara_\351\235\222\343\201\204\343\203\220\343\203\251/frimware/aoi_bara/config.h" 	modified:   "aoi bara_\351\235\222\343\201\204\343\203\220\343\203\251/frimware/aoi_bara/rules.mk" 	new file:   "aoi bara_\351\235\222\343\201\204\343\203\220\343\203\251/pcb/pcb/#auto_saved_files#" 	new file:   "aoi bara_\351\235\222\343\201\204\343\203\220\343\203\251/pcb/pcb/_autosave-pcb.kicad_pcb" 	new file:   "aoi bara_\351\235\222\343\201\204\343\203\220\343\203\251/pcb/pcb/_autosave-pcb.kicad_sch" 	modified:   "aoi bara_\351\235\222\343\201\204\343\203\220\343\203\251/pcb/pcb/freerouting.dsn" 	new file:   "aoi bara_\351\235\222\343\201\204\343\203\220\343\203\251/pcb/pcb/pcb-backups/pcb-2023-12-03_214633.zip" 	new file:   "aoi bara_\351\235\222\343\201\204\343\203\220\343\203\251/pcb/pcb/pcb-backups/pcb-2023-12-03_215222.zip" 	new file:   "aoi bara_\351\235\222\343\201\204\343\203\220\343\203\251/pcb/pcb/pcb-backups/pcb-2023-12-03_220250.zip" 	new file:   "aoi bara_\351\235\222\343\201\204\343\203\220\343\203\251/pcb/pcb/pcb-backups/pcb-2023-12-03_221316.zip" 	new file:   "aoi bara_\351\235\222\343\201\204\343\203\220\343\203\251/pcb/pcb/pcb-backups/pcb-2023-12-03_222808.zip" 	new file:   "aoi bara_\351\235\222\343\201\204\343\203\220\343\203\251/pcb/pcb/pcb-backups/pcb-2023-12-03_224939.zip" 	modified:   "aoi bara_\351\235\222\343\201\204\343\203\220\343\203\251/pcb/pcb/pcb.kicad_pcb" 	modified:   "aoi bara_\351\235\222\343\201\204\343\203\220\343\203\251/pcb/pcb/pcb.kicad_pro" 	new file:   "aoi bara_\351\235\222\343\201\204\343\203\220\343\203\251/pcb/pcb/production.rar" 	new file:   "aoi bara_\351\235\222\343\201\204\343\203\220\343\203\251/pcb/pcb/production/pcb-B_Cu.gbr" 	new file:   "aoi bara_\351\235\222\343\201\204\343\203\220\343\203\251/pcb/pcb/production/pcb-B_Mask.gbr" 	new file:   "aoi bara_\351\235\222\343\201\204\343\203\220\343\203\251/pcb/pcb/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
Routing:
- net GND: track 2.85 -> 27.6 mm
Changed lines of the file:
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@@
       (outputformat 1)
       (mirror false)
-      (drillshape 1)
+      (drillshape 0)
       (scaleselection 1)
-      (outputdirectory "")
+      (outputdirectory "production/")
     )
   )
@@
   (gr_rect (start 56.675 98.165) (end 371 193.415)
     (stroke (width 0.1) (type default)) (fill none) (layer "Edge.Cuts"))
-  (dimension (type aligned) (layer "F.Cu")
-    (pts (xy 371 98.165) (xy 371 193.415))
-    (height -23.69)
-    (gr_text "95.2500 mm" (at 392.89 145.79 90) (layer "F.Cu")
-      (effects (font (size 1.5 1.5) (thickness 0.3)))
-    )
-    (format (prefix "") (suffix "") (units 3) (units_format 1) (precision 4))
-    (style (thickness 0.2) (arrow_length 1.27) (text_position_mode 0) (extension_height 0.58642) (extension_offset 0.5) keep_text_aligned)
-  )
-  (dimension (type aligned) (layer "F.Cu")
-    (pts (xy 56.675 98.165) (xy 371 98.165))
-    (height -47.125)
-    (gr_text "314.3250 mm" (at 213.8375 49.24) (layer "F.Cu")
-      (effects (font (size 1.5 1.5) (thickness 0.3)))
-    )
-    (format (prefix "") (suffix "") (units 3) (units_format 1) (precision 4))
-    (style (thickness 0.2) (arrow_length 1.27) (text_position_mode 0) (extension_height 0.58642) (extension_offset 0.5) keep_text_aligned)
-  )
   (segment (start 75.341 105.14) (end 76.5225 105.14) (width 0.25) (layer "F.Cu") (net 1))
   (segment (start 267.0225 105.14) (end 286.0725 105.14) (width 0.25) (layer "F.Cu") (net 1))
@@
   (segment (start 357.92 130.32) (end 357.92 135.07) (width 0.25) (layer "B.Cu") (net 71))
   (segment (start 369.525 123.89) (end 369.05 123.89) (width 0.45) (layer "F.Cu") (net 72))
+  (segment (start 361.475 169.815) (end 361.475 163.195) (width 0.45) (layer "F.Cu") (net 72))
+  (segment (start 361.475 163.195) (end 355.44 157.16) (width 0.45) (layer "F.Cu") (net 72))
   (segment (start 366.705 130.045) (end 364.33 130.045) (width 0.45) (layer "F.Cu") (net 72))
+  (segment (start 355.44 157.16) (end 355.44 147.595) (width 0.45) (layer "F.Cu") (net 72))
   (segment (start 367.77 155.4) (end 367.77 138.565) (width 0.25) (layer "B.Cu") (net 73))
   (segment (start 358.975 155.315) (end 361.61 157.95) (width 0.25) (layer "B.Cu") (net 73))
@@
     (polygon
       (pts
-        (xy 56.675 98.165)
-        (xy 371 98.165)
-        (xy 371 193.415)
-        (xy 56.68 193.41)
+        (xy 57 98.5)
+        (xy 370.5 98.5)
+        (xy 370.8 193.21)
+        (xy 57 193)
       )
     )
