File: aoi bara_青いバラ/pcb/pcb/pcb.kicad_pcb (KiCad board)
At the start: 2 copper layers, 314.3 x 95.2 mm, 136 parts, among them J1 OLED_128x64, U1 Raspberry_Pi_Pico

Commit message: deleted:    "aoi bara_\351\235\222\343\201\204\343\203\220\343\203\251/pcb/pcb/#auto_saved_files#" 	deleted:    "aoi bara_\351\235\222\343\201\204\343\203\220\343\203\251/pcb/pcb/_autosave-pcb.kicad_pcb" 	deleted:    "aoi bara_\351\235\222\343\201\204\343\203\220\343\203\251/pcb/pcb/_autosave-pcb.kicad_sch" 	deleted:    "aoi bara_\351\235\222\343\201\204\343\203\220\343\203\251/pcb/pcb/pcb-backups/pcb-2023-11-17_233023.zip" 	new file:   "aoi bara_\351\235\222\343\201\204\343\203\220\343\203\251/pcb/pcb/pcb-backups/pcb-2024-01-28_124537.zip" 	modified:   "aoi bara_\351\235\222\343\201\204\343\203\220\343\203\251/pcb/pcb/pcb.kicad_pcb" 	modified:   "aoi bara_\351\235\222\343\201\204\343\203\220\343\203\251/pcb/pcb/pcb.kicad_prl" 	modified:   "aoi bara_\351\235\222\343\201\204\343\203\220\343\203\251/pcb/pcb/pcb.kicad_pro" 	modified:   "aoi bara_\351\235\222\343\201\204\343\203\220\343\203\251/pcb/pcb/pcb.kicad_sch" 	modified:   "aoi bara_\351\235\222\343\201\204\343\203\220\343\203\251/pcb/pcb/production/pcb-B_Cu.gbr" 	modified:   "aoi bara_\351\235\222\343\201\204\343\203\220\343\203\251/pcb/pcb/production/pcb-B_Mask.gbr" 	modified:   "aoi bara_\351\235\222\343\201\204\343\203\220\343\203\251/pcb/pcb/production/pcb-B_Paste.gbr" 	modified:   "aoi bara_\351\235\222\343\201\204\343\203\220\343\203\251/pcb/pcb/production/pcb-B_Silkscreen.gbr" 	modified:   "aoi bara_\351\235\222\343\201\204\343\203\220\343\203\251/pcb/pcb/production/pcb-Edge_Cuts.gbr" 	modified:   "aoi bara_\351\235\222\343\201\204\343\203\220\343\203\251/pcb/pcb/production/pcb-F_Cu.gbr" 	modified:   "aoi bara_\351\235\222\343\201\204\343\203\220\343\203\251/pcb/pcb/production/pcb-F_Mask.gbr" 	modified:   "aoi bara_\351\235\222\343\201\204\343\203\220\343\203\251/pcb/pcb/production/pcb-F_Paste.gbr" 	modified:   "aoi bara_\351\235\222\343\201\204\343\203\220\343\203\251/pcb/pcb/production/pcb-F_Silkscreen.gbr" 	modified:   "aoi bara_\351\235\222\343\201\204\343\203\220\343\203\251/pcb/pcb/production/pcb-NP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
Parts:
- added BZ1: Buzzer, Buzzer_Beeper:Buzzer_12x9.5RM7.6, B.Cu at (350.4, 155.9)
Connections:
- U1 pad 34: LED_DI -> Buzz
Routing:
- net Buzz: track 0.00 -> 53.9 mm, vias 0 -> 1
- net ROW4: track 377.1 -> 379.6 mm
- net en_co_A: track 50.9 -> 51.8 mm
- net COL10: track 183.9 -> 184.4 mm
Other:
- board size 314.3 x 95.2 mm -> 315 x 95.5 mm
